File: BPS-PowerPCB.kicad_sch (KiCad schematic)
At the start: 5 parts, among them J1 Conn_01x02, J2 Conn_01x02, J3 Conn_01x02, J4 Conn_01x02, J5 Conn_01x02

Commit message: done may need to add labels
Parts:
- removed J3, J4, J5: Conn_01x02, UTSVT_Connectors:Molex_MicroFit3.0_1x2xP3.00mm_PolarizingPeg_Vertical, symbol Connector_Generic:Conn_01x02
- added J3, J4, J5: Conn_01x04, Connector_Molex:Molex_Micro-Fit_3.0_43650-0415_1x04_P3.00mm_Vertical, symbol Connector_Generic:Conn_01x04
Connections:
- net +12V: now also J3.1 (Pin_1), J4.1 (Pin_1), J5.1 (Pin_1)
- net GND: now also J3.2 (Pin_2), J4.2 (Pin_2), J5.2 (Pin_2)
- no-connect marks 0 -> 6
